File: distributed_accel_quad.sch (KiCad schematic (older format))
At the start: 8 parts, among them U1 Teensy3.6, U2 CD74HC4067M, U3 MPU-9250

Commit message: Removed some resistors that aren't needed
Connections:
- wire segments 48 -> 47
Changed lines of the file:
@@
 Wire Wire Line
 	7250 2800 7250 3100
-Text GLabel 8100 2200 2    50   Input ~ 0
-3.3V
-Wire Wire Line
-	7950 2200 8100 2200
 Wire Wire Line
 	7950 2100 8500 2100
